Commit message: Add test_slam.sh
- Remove rviz from world.launch
- Rename robot_footprint to base_footprint to match gmapping default

File: home_service/urdf/my_robot.xacro (robot description, xacro)
@@ -2,8 +2,8 @@
 <robot name="my_robot" xmlns:xacro="http://www.ros.org/wiki/xacro">
   <xacro:include filename="$(find home_service)/urdf/my_robot.gazebo" />
-  <link name="robot_footprint"></link>
-  <joint name="robot_footprint_joint" type="fixed">
+  <link name="base_footprint"></link>
+  <joint name="base_footprint_joint" type="fixed">
     <origin xyz="0 0 0" rpy="0 0 0" />
-    <parent link="robot_footprint" />
+    <parent link="base_footprint" />
     <child link="chassis" />
   </joint>
